Commit message: fix: align calf folded pose limits
Set all four calf hard ranges to [-162, -48] degrees in the canonical URDF and generated MuJoCo models.

Keep position actuator targets aligned with the calf joint range, add a regression contract test, and document the separate RL soft safety range.

File: ros2/src/custom_dog_description/urdf/custom_dog.urdf (robot description, URDF)
Before this commit: robot custom_dog, 17 links, 16 joints
Joints:
- joint FL_calf_joint: limit lower=-2.7227 upper=-0.83776 effort=45 velocity=15 -> lower=-2.8274333882 upper=-0.83775804096 effort=45 velocity=15
- joint FR_calf_joint: limit lower=-2.7227 upper=-0.83776 effort=45 velocity=15 -> lower=-2.8274333882 upper=-0.83775804096 effort=45 velocity=15
- joint RL_calf_joint: limit lower=-2.7227 upper=-0.83776 effort=45 velocity=15 -> lower=-2.8274333882 upper=-0.83775804096 effort=45 velocity=15
- joint RR_calf_joint: limit lower=-2.7227 upper=-0.83776 effort=45 velocity=15 -> lower=-2.8274333882 upper=-0.83775804096 effort=45 velocity=15

Commit message: feat: consolidate locomotion pipeline and validation tooling
汇总当前 custom_dog_stack 的全向运动控制、恢复能力和跨物理验证工作。

主要内容：

- 完善闭环速度反馈、历史观测、课程采样、站立姿态、低速抬脚、步态鲁棒性和能耗/动作平滑相关配置。

- 修正纯角速度命令被误判为静止的站立奖励逻辑，并补充奖励、对称性、终止条件和训练器配置。

- 增加选择性自碰撞 URDF、MuJoCo 接触物理校验，以及跨 Isaac/MuJoCo 的策略轨迹、速度跟踪、机身姿态和恢复交接评测工具。

- 增加地形课程、闭环教师训练、213 维历史蒸馏、鲁棒站立、独立起身/自恢复和候选模型筛选脚本。

- 更新 sim2sim、键盘遥操作、候选导出、部署状态机、ROS 2 控制器和策略契约文档。

- 纳入当前评测报告、接触参数扫描结果和回归测试，覆盖训练脚本、评测脚本、MJCF/URDF 生成和策略控制接口。

- 忽略 ROS 构建产物及第三方依赖工作区，保留第三方 Dog-control 子仓库的本地未提交状态不变。

File: ros2/src/custom_dog_description/urdf/custom_dog.urdf (robot description, URDF)
Before this commit: robot custom_dog, 17 links, 16 joints
Links:
- link FL_calf: geometry collision cylinder length=0.185 radius=0.018; visual mesh filename=package://custom_dog_description/meshes/FL_calf.STL
- link FL_foot: geometry collision sphere radius=0.026; visual mesh filename=package://custom_dog_description/meshes/FL_foot.STL
- link FL_hip: geometry collision cylinder length=0.090 radius=0.040; visual mesh filename=package://custom_dog_description/meshes/FL_hip.STL
- link FL_thigh: geometry collision cylinder length=0.190 radius=0.035; visual mesh filename=package://custom_dog_description/meshes/FL_thigh.STL
- link FR_calf: geometry collision cylinder length=0.185 radius=0.018; visual mesh filename=package://custom_dog_description/meshes/FR_calf.STL
- link FR_foot: geometry collision sphere radius=0.026; visual mesh filename=package://custom_dog_description/meshes/FR_foot.STL
- link FR_hip: geometry collision cylinder length=0.090 radius=0.040; visual mesh filename=package://custom_dog_description/meshes/FR_hip.STL
- link FR_thigh: geometry collision cylinder length=0.190 radius=0.035; visual mesh filename=package://custom_dog_description/meshes/FR_thigh.STL
- link RL_calf: geometry collision cylinder length=0.185 radius=0.018; visual mesh filename=package://custom_dog_description/meshes/RL_calf.STL
- link RL_foot: geometry collision sphere radius=0.026; visual mesh filename=package://custom_dog_description/meshes/RL_foot.STL
- link RL_hip: geometry collision cylinder length=0.090 radius=0.040; visual mesh filename=package://custom_dog_description/meshes/RL_hip.STL
- link RL_thigh: geometry collision cylinder length=0.190 radius=0.035; visual mesh filename=package://custom_dog_description/meshes/RL_thigh.STL
- link RR_calf: geometry collision cylinder length=0.185 radius=0.018; visual mesh filename=package://custom_dog_description/meshes/RR_calf.STL
- link RR_foot: geometry collision sphere radius=0.026; visual mesh filename=package://custom_dog_description/meshes/RR_foot.STL
- link RR_hip: geometry collision cylinder length=0.090 radius=0.040; visual mesh filename=package://custom_dog_description/meshes/RR_hip.STL
- link RR_thigh: geometry collision cylinder length=0.190 radius=0.035; visual mesh filename=package://custom_dog_description/meshes/RR_thigh.STL
- link base: geometry collision box size=0.255 0.220 0.100; visual mesh filename=package://custom_dog_description/meshes/base.STL
