Commit message: fix(asset): separate collision contracts by simulator
Keep custom_dog.urdf as the complete canonical robot model with collision geometry on all 17 links. Regenerate the calibrated Isaac proxy asset, add a deterministic Gazebo point-foot generator and checked-in URDF that removes exactly the eight thigh/calf ground colliders, and switch the legacy Isaac configuration to the calibrated proxy. Add regression tests for canonical, Isaac, and Gazebo variants, extend static validation, and advance Dog-control to the launch-time model-selection implementation. This prevents simulator workarounds from mutating the shared robot description.

File: ros2/src/custom_dog_description/urdf/custom_dog_gazebo_point_foot.urdf (robot description, URDF)
Before this commit: robot custom_dog, 17 links, 16 joints
Links:
- link FL_calf: geometry visual mesh filename=package://custom_dog_description/meshes/FL_calf.STL
- link FL_thigh: geometry visual mesh filename=package://custom_dog_description/meshes/FL_thigh.STL
- link FR_calf: geometry visual mesh filename=package://custom_dog_description/meshes/FR_calf.STL
- link FR_thigh: geometry visual mesh filename=package://custom_dog_description/meshes/FR_thigh.STL
- link RL_calf: geometry visual mesh filename=package://custom_dog_description/meshes/RL_calf.STL
- link RL_thigh: geometry visual mesh filename=package://custom_dog_description/meshes/RL_thigh.STL
- link RR_calf: geometry visual mesh filename=package://custom_dog_description/meshes/RR_calf.STL
- link RR_thigh: geometry visual mesh filename=package://custom_dog_description/meshes/RR_thigh.STL
